File: Tesi.kicad_sch (KiCad schematic)
At the start: 0 parts

Commit message: Project started
Parts:
- added C11: ~, Capacitor_SMD:C_0603_1608Metric, symbol Device:C
- added IC1: STM32G474RET6, QFP50P1200X1200X160-64N, symbol STM32G474RET6:STM32G474RET6
- added J1: Conn_ST_STDC14, symbol Connector:Conn_ST_STDC14
- added Q1: FDS8858CZ, SOIC127P600X175-8N, symbol FDS8858CZ:FDS8858CZ
- added SW2: reset, Button_Switch_SMD:SW_SPST_FSMSM, symbol Switch:SW_Push
- added U1: LD1117S33TR_SOT223, Package_TO_SOT_SMD:SOT-223-3_TabPin2, symbol Regulator_Linear:LD1117S33TR_SOT223
Connections:
- new net: J1.5 (GND), J1.7 (GND)
- new net GND: C11.2, SW2.2
- new net NRST: C11.1, SW2.1

Commit message: first commit. added some symbols
Parts:
- added C1, C2, C4, C5, C6: C, symbol Device:C
- added C3: C_Polarized, symbol Device:C_Polarized
- added D1, D2, D4: SP4020-01FTG-C, SOD2613X114N, symbol SP4020-01FTG-C:SP4020-01FTG-C
- added D3: D, symbol Device:D
- added IC2: NDC7002N, SOT95P275X110-6N, symbol NDC7002N:NDC7002N
- added IC3: TLC272BCDR, SOIC127P600X175-8N, symbol TLC272BCDR:TLC272BCDR
- added J2: MSS-102545-14A-D, MSS10254514AD, symbol MSS-102545-14A-D:MSS-102545-14A-D
- added J3: S2B-PH-K-S_LF__SN_, SHDRRA2W50P0X200_1X2_590X760X480P, symbol S2B-PH-K-S_LF__SN_:S2B-PH-K-S_LF__SN_
- added L1: L, symbol Device:L
- added Q2: PMOS, symbol Simulation_SPICE:PMOS
- added R1, R2, R3: R, symbol Device:R
- added U2: ${SIM.PARAMS}, symbol Simulation_SPICE:OPAMP
Connections:
- net GND: now also U1.1 (GND), C1.2, C2.2, C3.2, C4.2, C5.2, C6.2, D1.1, D2.1, D3.2 (A), D4.1, IC3.4 (GND), R2.2
- net +3V3: now reaches U1.2 (VO)
- net +3V3: now also C1.1, C6.1, D4.2, IC3.8 (VDD)
- net at U1.3 (VI): now also C5.1
- new net: D3.1 (K), L1.1, Q2.1 (D)
- new net: C3.1, L1.2
- new net: C2.1, D1.2, IC3.3 (1IN+), R1.2, R2.1
- new net BUCK_CTRL: D2.2, Q2.2 (G)
- new net HV: R1.1
- new net PID: IC3.1 (1OUT), IC3.2 (1IN-)
- new net VBUCK: C4.1, Q2.3 (S)
- no-connect marks 0 -> 3
Other:
- note added: "Buck & FB"
- moved on the sheet: Q1, U1

Commit message: Updated Schematic
Parts:
- added C10, C7, C8, C9: C, symbol Device:C
- added D10: D, symbol Device:D
- added D11, D12: SP4020-01FTG-C, SOD2613X114N, symbol SP4020-01FTG-C:SP4020-01FTG-C
- added D5, D7, D8: LED, symbol Device:LED
- added D6, D9: ~, symbol Sensor_Optical:BP104-SMD
- added IC4: NDC7002N, SOT95P275X110-6N, symbol NDC7002N:NDC7002N
- added J4: S2B-PH-K-S_LF__SN_, SHDRRA2W50P0X200_1X2_590X760X480P, symbol S2B-PH-K-S_LF__SN_:S2B-PH-K-S_LF__SN_
- added J5: MSS-102545-14A-D, MSS10254514AD, symbol MSS-102545-14A-D:MSS-102545-14A-D
- added Q3, Q4, Q5, Q6: Q_NMOS_SGD, symbol Transistor_FET:Q_NMOS_SGD
- added R10, R11, R4, R5, R6, R7, R8, R9: R, symbol Device:R
Connections:
- net +3V3: now also C10.1, R10.1, R11.1
- net GND: now also J2.3 (NC), C10.2, C7.2, C8.2, C9.2, D11.1, D12.1, D9.2 (A), J4.2, J5.3 (NC), Q3.1 (S), Q4.1 (S), Q5.1 (S), Q6.1 (S), R4.2
- net HV: now also D10.2 (A)
- net VBUCK: now also J5.2 (NO)
- net VIN: now also J2.2 (NO), C8.1, D5.2 (A), R5.1, R6.1
- net VBATT: now reaches J2.1 (COM)
- net VBATT: now also J3.1
- net at J3.2: now also J4.1
- new net: D5.1 (K), R7.1
- new net: D7.1 (K), R8.1
- new net: Q3.3 (D), Q4.2 (G), R6.2
- new net: C7.1, Q3.2 (G), R4.1, R5.2
- new net: D8.1 (K), R9.1
- new net: Q6.3 (D), R9.2
- new net: D12.2, Q6.2 (G), R10.2
- new net: D11.2, Q5.2 (G), R11.2
- new net: Q5.3 (D), R8.2
- new net: Q4.3 (D), R7.2
- new net: D10.1 (K), D6.1 (K)
- new net +5V: C9.1, D7.2 (A), D8.2 (A), J5.1 (COM)
- new net HVOUT-X: D6.2 (A), D9.1 (K)
Other:
- note added: "Battery & Power"
- note added: "Channel Control"
- moved on the sheet: C1, C11, C2, C3, C4, C5, C6, D1, D2, D3, D4, IC1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

Commit message: MCU CubeMX Project
Parts:
- removed IC1: STM32G474RET6, QFP50P1200X1200X160-64N, symbol STM32G474RET6:STM32G474RET6
- added C12: 4.7uF, Capacitor_SMD:C_0603_1608Metric, symbol Device:C
- added C13: 100nF, Capacitor_SMD:C_0603_1608Metric, symbol Device:C
- added C14, C15: 18p, Capacitor_SMD:C_0603_1608Metric, symbol Device:C
- added D13: LED, symbol Device:LED
- added R12: R, symbol Device:R
- added U3: STM32C092FCP6, symbol Eagle_Main:STM32C092FCP6
- added Y2: X_MHz, Crystal:Crystal_SMD_3225-4Pin_3.2x2.5mm, symbol Device:Crystal_GND24_Small
- J1: footprint (none) -> Eagle_Connectors:SAMTEC_FTSH-107-01-L-DV-K-TR
Connections:
- net +3V3: now also J1.3 (VCC), C12.1, C13.1, U3.4 (VDD/VDDA)
- net GND: now also J1.11 (GNDDetect), J1.5 (GND), J1.7 (GND), C12.2, C13.2, C14.2, C15.2, D13.1 (K), U3.5 (VSS/VSSA), Y2.2, Y2.4
- net NRST: now also J1.12 (~{RST}), U3.6 (PF2-NRST)
- net PID: now also U3.9 (PA2)
- net RX_SWD: now reaches J1.13 (VCP_RX)
- net RX_SWD: now also U3.8 (PA1)
- net TX_SWD: now reaches J1.14 (VCP_TX)
- net TX_SWD: now also U3.7 (PA0)
- net SWDIO: now reaches J1.4 (JTMS/SWDIO)
- net SWDIO: now also U3.18 (PA13)
- net SWCLK: now reaches J1.6 (JCLK/SWCLK)
- net SWCLK: now also U3.19 (PA14-BOOT0/PA15)
- new net: D13.2 (A), R12.2
- new net OSC_IN: C14.1, U3.2 (PC14-OSCX_IN), Y2.1
- new net OSC_OUT: C15.1, U3.3 (PC15-OSCX_OUT), Y2.3
- new net USER_LED: R12.1, U3.16 (PA11[PA9])
- no-connect marks 3 -> 6
Other:
- note added: "5V"
- note added: "Debug Connector"
- note added: "Decupling"
- note added: "Oscillator"
- note added: "Place as close as possible VDD and VSS pins"
- moved on the sheet: C1, C10, C11, C2, C3, C4, C5, C6, C7, C8, C9, D1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

Commit message: added some comments about future jobs
Parts:
- added J6: Conn_01x01_Socket, symbol Connector:Conn_01x01_Socket
Connections:
- net HVOUT-X: now also J6.1 (Pin_1)
Other:
- note added: "- Quanti canali mettere - Trovare simbolo e Footprint del componente mancante nella parte di buck, magari adattando quelle di un modello simile che ho trovato in rete -Trovare un regolatore di tensione equivalente al D24V50F5 usato nella parte di Power, oppure trovare il modo di integrarlo nella pcb -simulare qualche parte su spice ? -i simboli degli integrati usati nel progetto conteneti mosfet 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"
- note added: "MCU"
- moved on the sheet: C11, C12, C13, C14, C15, D13, J1, R12, R3, SW2, U3, Y2
